Commit message: Updated Nextore gazebo simulations

File: src/working/models/3DLidar/3d_lidar_truck.xacro (robot description, xacro)
@@ -50,5 +50,5 @@
     <visual>
         <geometry>
-          <mesh filename="package://working/models/Truck/180tonnes_v4.dae"/>
+          <mesh filename="package://working/models/Truck/MR_Roboto.dae"/>
         </geometry>
         <origin xyz="0 0 0" rpy="0 0 0" />
@@ -56,5 +56,5 @@
     <collision>
         <geometry>
-          <mesh filename="package://working/models/Truck/180tonnes_v4.dae"/>
+          <mesh filename="package://working/models/Truck/MR_Roboto.dae"/>
         </geometry>
         <origin xyz="0 0 0" rpy="0 0 0" />
@@ -119,5 +119,5 @@
 <joint name="3d_lidar_joint" type="fixed">
     <axis xyz="0 1 0"/>
-    <origin rpy="0 ${M_PI/2} 0" xyz="0 0 10"/>
+    <origin rpy="0 ${M_PI/2} 0" xyz="0 0 8"/>
     <parent link="base_footprint"/>
     <child link="3d_lidar"/>
@@ -161,5 +161,5 @@
 <joint name="camera_link_joint" type="fixed">
     <axis xyz="0 1 0"/>
-    <origin rpy="0 ${M_PI/2} 0" xyz="0.2 0 10"/>
+    <origin rpy="0 ${M_PI/2} 0" xyz="1 0 7"/>
     <parent link="base_footprint"/>
     <child link="camera_link"/>
