Commit message: Added code to accumulate exscan point cloud overtime

File: src/working/models/3DLidar/3d_lidar_flashlights_and_trucks_drive_in.xacro (robot description, xacro)
@@ -726,3 +726,85 @@
     </actuator>
   </transmission>
+    <!-- Camera addition -->
+     <link name="camera_link_front">
+        <visual>
+            <origin xyz="0.0149 0.0 0.0125" rpy="${M_PI/2} 0 ${M_PI/2}"/>
+            <geometry>
+                <mesh filename="package://realsense2_description/meshes/d435.dae" />
+            </geometry>
+            <material name="Neobotix/Aluminum"/>
+        </visual>
+        <collision>
+            <origin xyz="0.0149 0.0 0.0125" rpy="${M_PI/2} 0 ${M_PI/2}"/>
+            <geometry>
+                <box size="0.02505 0.09 0.025"/>
+            </geometry>
+        </collision>
+        <inertial>
+            <mass value="0.564" />
+            <origin xyz="0.0149 0.0 0.0125" rpy="${M_PI/2} 0 ${M_PI/2}"/>
+            <inertia ixx="0.003881243" ixy="0.0" ixz="0.0" iyy="0.000498940" iyz="0.0" izz="0.003879257" />
+        </inertial>
+    </link>
+    <joint name="camera_joint_front" type="fixed">
+        <origin xyz="0.23 0 0.13" rpy="0 0 0"/>
+        <axis xyz="0 1 0"/>
+        <parent link="base_link"/>
+        <child link="camera_link_front"/>
+    </joint>
+    <link name="camera_depth_frame_front"/>
+    <joint name="camera_depth_joint_front" type="fixed">
+        <origin xyz="0 0 0" rpy="${-M_PI/2} 0 ${-M_PI/2}" />
+        <parent link="camera_link_front" />
+        <child link="camera_depth_frame_front" />
+    </joint>
+    <gazebo reference="camera_link_front">
+        <sensor type="depth" name="sensor_d435">
+            <visualize>true</visualize>
+            <update_rate>24</update_rate>
+            <camera>
+                <horizontal_fov>1.3962634</horizontal_fov>
+                <image>
+                    <format>B8G8R8</format>
+                    <!-- HD 1080 x 720 -->
+                    <!-- SD  640 x 480 -->
+                    <!-- LD  320 x 240 -->
+                    <width>1080</width>
+                    <height>720</height>
+                </image>
+                <clip>
+                    <near>0.15</near>
+                    <far>20</far>
+                </clip>
+                <noise>
+                    <type>gaussian</type>
+                    <mean>0.0</mean>
+                    <stddev>0.007</stddev>
+                </noise>
+            </camera>
+            <plugin name="sensor_d435_controller" filename="libgazebo_ros_openni_kinect.so">
+                <baseline>0.2</baseline>
+                <alwaysOn>true</alwaysOn>
+                <updateRate>0.0</updateRate>
+                <cameraName>sensor_d435_front</cameraName>
+                <imageTopicName>/sensor_d435_front/image_raw</imageTopicName>
+                <cameraInfoTopicName>/sensor_d435_front/color/camera_info</cameraInfoTopicName>
+                <depthImageTopicName>/sensor_d435_front/depth/image_rect_raw</depthImageTopicName>
+                <depthImageInfoTopicName>/sensor_d435_front/depth/camera_info</depthImageInfoTopicName>
+                <pointCloudTopicName>/sensor_d435_front/depth/points</pointCloudTopicName>
+                <frameName>camera_depth_frame_front</frameName>
+                <pointCloudCutoff>0.0</pointCloudCutoff>
+                <distortionK1>0.00000001</distortionK1>
+                <distortionK2>0.00000001</distortionK2>
+                <distortionK3>0.00000001</distortionK3>
+                <distortionT1>0.00000001</distortionT1>
+                <distortionT2>0.00000001</distortionT2>
+                <CxPrime>0</CxPrime>
+                <Cx>0</Cx>
+                <Cy>0</Cy>
+                <focalLength>0.0</focalLength>
+                <hackBaseline>0.0</hackBaseline>
+            </plugin>
+        </sensor>
+    </gazebo>
 </robot>
